File: Pro_Rev2/Pro_Rev2.kicad_sch (KiCad schematic)
At the start: 279 parts, among them J1 USB_C_Receptacle, J10 IO28, J11 GP27_R, J12 GP28_R, J13 TP1, J14 TP2, J2 AudioJack4, J3 OLED, J4 TP1, J5 TP2, J6 USB_C_Receptacle, J7 OLED, J8 AudioJack4, J9 IO27, SW1 SW_Push, SW10 SW_Push, SW11 SW_Push, SW12 SW_Push, SW13 SW_Push, SW14 SW_Push, SW15 SW_Push, SW16 SW_Push, SW17 SW_Push, SW18 SW_Push, SW19 SW_Push, SW2 SW_Push, SW20 SW_Push, SW21 SW_Push, SW22 SW_Push, SW23 SW_Push, SW24 SW_Push, SW25 SW_Push, SW26 SW_Push, SW27 SW_Push, SW28 SW_Push, SW29 SW_Push, SW3 SW_Push, SW30 SW_Push, SW31 SW_Push, SW32 SW_Push, SW33 SW_Push, SW34 SW_Push, SW35 SW_Push, SW36 SW_Push, SW37 SW_Push, SW38 SW_Push, SW39 SW_Push, SW4 SW_Push, SW40 SW_Push, SW41 SW_Push, SW42 SW_Push, SW43 SW_Push, SW44 SW_Push, SW45 SW_Push, SW46 SW_Push, SW47 SW_Push, SW48 SW_Push, SW49 SW_Push, SW5 SW_Push, SW50 SW_Push, SW51 SW_Push, SW52 SW_Push, SW53 SW_Push, SW54 SW_Push, SW55 SW_Push, SW56 SW_Push, SW57 SW_Push, SW58 SW_Push, SW6 SW_Push, SW7 SW_Push, SW8 SW_Push, SW9 SW_Push, U1 NCP1117-3.3_SOT223, U2 USBLC6-2SC6, U3 RP2040, U4 W25Q128JVPIQ, U5 NCP1117-3.3_SOT223, U6 USBLC6-2SC6, U7 RP2040, U8 W25Q128JVPIQ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

Commit message: add Lily58 Pro Rev2 PCB
Parts:
- removed RE1: Rotary_Encoder_Switch, KiCad:RotaryEncoder_Alps_EC11E-Switch_Vertical_H20mm_CircularMountingHoles, symbol Device:Rotary_Encoder_Switch
- R1, R10: value 1k -> 50k
Connections:
- net COL0_R: now also SW35.1, SW41.1, SW47.1, SW53.1, U7.7 (GPIO5); no longer SW30.1, SW36.1, SW42.1, SW48.1, SW54.1, U7.13 (GPIO10)
- net COL1_R: now also SW34.1, SW40.1, SW46.1, SW52.1, SW58.1, U7.8 (GPIO6); no longer SW31.1, SW37.1, SW43.1, SW49.1, SW55.1, U7.12 (GPIO9)
- net COL2_R: now also SW33.1, SW39.1, SW45.1, SW51.1, SW57.1, U7.9 (GPIO7); no longer SW32.1, SW38.1, SW44.1, SW50.1, SW56.1, U7.11 (GPIO8)
- net COL3_R: now also SW32.1, SW38.1, SW44.1, SW50.1, SW56.1, U7.11 (GPIO8); no longer SW33.1, SW39.1, SW45.1, SW51.1, SW57.1, U7.9 (GPIO7)
- net COL4_R: now also SW31.1, SW37.1, SW43.1, SW49.1, SW55.1, U7.12 (GPIO9); no longer SW34.1, SW40.1, SW46.1, SW52.1, SW58.1, U7.8 (GPIO6)
- net COL5_R: now also SW30.1, SW36.1, SW42.1, SW48.1, SW54.1, U7.13 (GPIO10); no longer SW35.1, SW41.1, SW47.1, SW53.1, U7.7 (GPIO5)
- net LED: now also LED6.4 (DIN); no longer LED1.4 (DIN)
- net LED_R: now also LED35.4 (DIN); no longer LED30.4 (DIN)
- net at LED6.2 (DOUT): now also LED5.4 (DIN); no longer LED12.4 (DIN)
- net at LED5.2 (DOUT): now also LED4.4 (DIN); no longer LED6.4 (DIN)
- net at LED54.2 (DOUT): no longer LED55.4 (DIN)
- net at LED54.4 (DIN): now also LED55.2 (DOUT); no longer LED48.2 (DOUT)
- net at LED21.2 (DOUT): now also LED22.4 (DIN); no longer LED20.4 (DIN)
- net at LED21.4 (DIN): now also LED20.2 (DOUT); no longer LED22.2 (DOUT)
- net at LED37.2 (DOUT): now also LED38.4 (DIN); no longer LED36.4 (DIN)
- net at LED37.4 (DIN): now also LED36.2 (DOUT); no longer LED38.2 (DOUT)
- net at LED30.2 (DOUT): now also LED36.4 (DIN); no longer LED31.4 (DIN)
- net at LED45.2 (DOUT): now also LED44.4 (DIN); no longer LED46.4 (DIN)
- net at LED45.4 (DIN): now also LED46.2 (DOUT); no longer LED44.2 (DOUT)
- net at LED52.2 (DOUT): now also LED53.4 (DIN); no longer LED51.4 (DIN)
- net at LED52.4 (DIN): now also LED51.2 (DOUT); no longer LED53.2 (DOUT)
- net at LED19.4 (DIN): now also LED13.2 (DOUT); no longer LED20.2 (DOUT)
- net at LED58.2 (DOUT): now also LED57.4 (DIN)
- net at LED58.4 (DIN): now also LED53.2 (DOUT); no longer LED57.2 (DOUT)
- net at LED19.2 (DOUT): now also LED20.4 (DIN); no longer LED25.4 (DIN)
- net at LED14.2 (DOUT): now also LED13.4 (DIN); no longer LED15.4 (DIN)
- net at LED14.4 (DIN): now also LED15.2 (DOUT); no longer LED13.2 (DOUT)
- net at LED56.2 (DOUT): now also LED55.4 (DIN); no longer LED57.4 (DIN)
- net at LED56.4 (DIN): now also LED57.2 (DOUT); no longer LED55.2 (DOUT)
- net at LED8.2 (DOUT): now also LED9.4 (DIN); no longer LED7.4 (DIN)
- net at LED8.4 (DIN): now also LED7.2 (DOUT); no longer LED9.2 (DOUT)
- net at LED41.2 (DOUT): now also LED47.4 (DIN); no longer LED40.4 (DIN)
- net at LED41.4 (DIN): now also LED40.2 (DOUT); no longer LED35.2 (DOUT)
- net at LED10.2 (DOUT): now also LED11.4 (DIN); no longer LED9.4 (DIN)
- net at LED10.4 (DIN): now also LED9.2 (DOUT); no longer LED11.2 (DOUT)
- net at LED42.4 (DIN): now also LED43.2 (DOUT); no longer LED36.2 (DOUT)
- net at LED50.2 (DOUT): now also LED51.4 (DIN); no longer LED49.4 (DIN)
- net at LED50.4 (DIN): now also LED49.2 (DOUT); no longer LED51.2 (DOUT)
- net at LED34.2 (DOUT): now also LED33.4 (DIN); no longer LED35.4 (DIN)
- net at LED48.4 (DIN): now also LED42.2 (DOUT); no longer LED49.2 (DOUT)
- net at LED1.2 (DOUT): now also LED7.4 (DIN); no longer LED2.4 (DIN)
- net at LED39.4 (DIN): now also LED38.2 (DOUT); no longer LED40.2 (DOUT)
- net at LED3.2 (DOUT): now also LED2.4 (DIN); no longer LED4.4 (DIN)
- net at LED2.2 (DOUT): now also LED1.4 (DIN); no longer LED3.4 (DIN)
- net at LED23.2 (DOUT): now also LED24.4 (DIN); no longer LED22.4 (DIN)
- net at LED23.4 (DIN): now also LED22.2 (DOUT); no longer LED24.2 (DOUT)
- net at LED16.2 (DOUT): now also LED15.4 (DIN); no longer LED17.4 (DIN)
- net at LED16.4 (DIN): now also LED17.2 (DOUT); no longer LED15.2 (DOUT)
- net at LED26.2 (DOUT): now also LED25.4 (DIN); no longer LED27.4 (DIN)
- net at LED26.4 (DIN): now also LED27.2 (DOUT); no longer LED25.2 (DOUT)
- net at LED18.2 (DOUT): now also LED17.4 (DIN); no longer LED24.4 (DIN)
- net at LED31.2 (DOUT): now also LED30.4 (DIN); no longer LED32.4 (DIN)
- net at LED4.2 (DOUT): now also LED3.4 (DIN); no longer LED5.4 (DIN)
- net at LED18.4 (DIN): now also LED12.2 (DOUT); no longer LED17.2 (DOUT)
- net at LED34.4 (DIN): now also LED35.2 (DOUT); no longer LED33.2 (DOUT)
- net at LED28.4 (DIN): now also LED29.2 (DOUT); no longer LED27.2 (DOUT)
- net at LED47.2 (DOUT): now also LED46.4 (DIN); no longer LED53.4 (DIN)
- net at LED29.4 (DIN): now also LED24.2 (DOUT); no longer LED28.2 (DOUT)
- net at LED39.2 (DOUT): now also LED40.4 (DIN); no longer LED38.4 (DIN)
- net at LED32.2 (DOUT): now also LED31.4 (DIN); no longer LED33.4 (DIN)
- net at LED43.4 (DIN): now also LED44.2 (DOUT); no longer LED42.2 (DOUT)
- net RE_A: no longer names the net of U3.5 (GPIO3)
- net RE_B: no longer names the net of U3.4 (GPIO2)
- net RE_SW: no longer names the net of D29.2 (A), SW29.2
- new net: LED48.2 (DOUT), LED49.4 (DIN)
- new net: LED11.2 (DOUT), LED12.4 (DIN)
- new net: LED27.4 (DIN), LED28.2 (DOUT)
- new net: LED32.4 (DIN), LED33.2 (DOUT)
- no-connect marks 44 -> 52
Other:
- note added: "I2D1 SCL"
- note added: "I2D1 SDA"
- note removed: "I2C0 SCL"
- note removed: "I2C0 SDA"
- moved on the sheet: LED1, LED10, LED11, LED12, LED13, LED14, LED15, LED16, LED17, LED18, LED19, LED2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

Commit message: Update Lily58 ProRev2
Parts:
- removed J13, J4: TP1, TestPoint:TestPoint_Pad_D1.0mm, symbol Connector:Conn_01x01_Male
- removed J14, J5: TP2, TestPoint:TestPoint_Pad_D1.0mm, symbol Connector:Conn_01x01_Male
- added TP1, TP12: TP_COL0, yuchi:TestPoint_Pad_1mm, symbol Connector:TestPoint
- added TP10, TP21: TP_ROW3, yuchi:TestPoint_Pad_1mm, symbol Connector:TestPoint
- added TP11, TP22: TP_ROW4, yuchi:TestPoint_Pad_1mm, symbol Connector:TestPoint
- added TP13, TP2: TP_COL1, yuchi:TestPoint_Pad_1mm, symbol Connector:TestPoint
- added TP14, TP3: TP_COL2, yuchi:TestPoint_Pad_1mm, symbol Connector:TestPoint
- added TP15, TP4: TP_COL3, yuchi:TestPoint_Pad_1mm, symbol Connector:TestPoint
- added TP16, TP5: TP_COL4, yuchi:TestPoint_Pad_1mm, symbol Connector:TestPoint
- added TP17, TP6: TP_COL5, yuchi:TestPoint_Pad_1mm, symbol Connector:TestPoint
- added TP18, TP7: TP_ROW0, yuchi:TestPoint_Pad_1mm, symbol Connector:TestPoint
- added TP19, TP8: TP_ROW1, yuchi:TestPoint_Pad_1mm, symbol Connector:TestPoint
- added TP20, TP9: TP_ROW2, yuchi:TestPoint_Pad_1mm, symbol Connector:TestPoint
- added TP23, TP25: SCL_2, yuchi:TestPoint_Pad_1mm, symbol Connector:TestPoint
- added TP24, TP26: SDA_2, yuchi:TestPoint_Pad_1mm, symbol Connector:TestPoint
- added TP27, TP30: SWD, yuchi:TestPoint_Pad_1mm, symbol Connector:TestPoint
- added TP28, TP31: GND, yuchi:TestPoint_Pad_1mm, symbol Connector:TestPoint
- added TP29, TP32: SWC, yuchi:TestPoint_Pad_1mm, symbol Connector:TestPoint
- C10, C13, C20, C25, C26, C5: footprint Capacitor_SMD:C_0402_1005Metric -> Capacitor_SMD:C_0603_1608Metric
- J10, J11, J12, J9: footprint TestPoint:TestPoint_Pad_D1.0mm -> yuchi:TestPoint_Pad_1mm
- Y1: value 12MHz_Q22FA23V00285 -> 12MHz
- Y2: value Crystal -> 12MHz
Connections:
- net COL0: now also TP1.1
- net COL0_R: now also TP12.1
- net COL1: now also TP2.1
- net COL1_R: now also TP13.1
- net COL2: now also TP3.1
- net COL2_R: now also TP14.1
- net COL3: now also TP4.1
- net COL3_R: now also TP15.1
- net COL4: now also TP5.1
- net COL4_R: now also TP16.1
- net COL5: now also TP6.1
- net COL5_R: now also TP17.1
- net GND: now also TP28.1
- net GNDA: now also TP31.1
- net ROW0: now also TP7.1
- net ROW0_R: now also TP18.1
- net ROW1: now also TP8.1
- net ROW1_R: now also TP19.1
- net ROW2: now also TP9.1
- net ROW2_R: now also TP20.1
- net ROW3: now also TP10.1
- net ROW3_R: now also TP21.1
- net ROW4: now also TP11.1
- net ROW4_R: now also TP22.1
- net SWCLK: now also TP29.1
- net SWCLK_R: now also TP32.1
- net SWD: now also TP27.1
- net SWD_R: now also TP30.1
- net SDA_2: now reaches U3.4 (GPIO2)
- net SDA_2: now also TP24.1
- net SCL_2: now reaches U3.5 (GPIO3)
- net SCL_2: now also TP23.1
- net SDA_2_R: now reaches U7.4 (GPIO2)
- net SDA_2_R: now also TP26.1
- net SCL_2_R: now reaches U7.5 (GPIO3)
- net SCL_2_R: now also TP25.1
- no-connect marks 52 -> 62
