File: Pro_V2/Pro_V2.kicad_sch (KiCad schematic)
At the start: 322 parts, among them J1 USB_C_Receptacle, J2 AudioJack4, J3 OLED, J6 USB_C_Receptacle, J7 OLED, J8 AudioJack4, SW1 SW_Push, SW10 SW_Push, SW11 SW_Push, SW12 SW_Push, SW13 SW_Push, SW14 SW_Push, SW15 SW_Push, SW16 SW_Push, SW17 SW_Push, SW18 SW_Push, SW19 SW_Push, SW2 SW_Push, SW20 SW_Push, SW21 SW_Push, SW22 SW_Push, SW23 SW_Push, SW24 SW_Push, SW25 SW_Push, SW26 SW_Push, SW27 SW_Push, SW28 SW_Push, SW29 SW_Push, SW3 SW_Push, SW30 SW_Push, SW31 SW_Push, SW32 SW_Push, SW33 SW_Push, SW34 SW_Push, SW35 SW_Push, SW36 SW_Push, SW37 SW_Push, SW38 SW_Push, SW39 SW_Push, SW4 SW_Push, SW40 SW_Push, SW41 SW_Push, SW42 SW_Push, SW43 SW_Push, SW44 SW_Push, SW45 SW_Push, SW46 SW_Push, SW47 SW_Push, SW48 SW_Push, SW49 SW_Push, SW5 SW_Push, SW50 SW_Push, SW51 SW_Push, SW52 SW_Push, SW53 SW_Push, SW54 SW_Push, SW55 SW_Push, SW56 SW_Push, SW57 SW_Push, SW58 SW_Push, SW6 SW_Push, SW7 SW_Push, SW8 SW_Push, SW9 SW_Push, U1 AMS1117-3.3, U10 TXB0104RUT, U2 USBLC6-2SC6, U3 RP2040, U4 W25Q128JVPIQ, U5 AMS1117-3.3, U6 USBLC6-2SC6, U7 RP2040, U8 W25Q128JVPIQ, U9 TXB0104RUT, Y1 12MHz, Y2 12MHz

Commit message: Pro v2 update
Other:
- title: (none) -> Lily58 Pro v2
